Commit message: Fixed package name fixed depency in r2d2 cleaning done

File: models/r2d4.urdf (robot description, URDF)
Before this commit: robot physics, 12 links, 11 joints
Links:
- link hokuyo_link: geometry collision box size=0.1 0.1 0.1; visual mesh filename=package://mapnplan/models/meshes/hokuyo.dae

Commit message: Robot goes out of the room

File: models/r2d4.urdf (robot description, URDF)
Before this commit: robot physics, 12 links, 11 joints
Links:
- added link head_ball, mass 0.00001; collision sphere radius=0.2; visual sphere radius=0.2
- added link head_ball_box, mass 0.00001; collision box size=.1 0.1 .1; visual box size=.1 0.1 .1
Joints:
- added joint head_ball_box_swivel: type fixed, parent head_ball, child head_ball_box, origin xyz=0 0.15 0.15 rpy=0 0 0, axis 0 0 1, limit effort=100 velocity=100
- added joint head_ball_swivel: type fixed, parent head, child head_ball, origin xyz=0 0 0.5 rpy=0 0 0, axis 0 0 1, limit effort=100 velocity=100
